Commit message: +rgbd camera +fixed rover tilt and zones

File: curiosity_description/models/urdf/sensor_mast.xacro (robot description, xacro)
@@ -234,4 +234,10 @@
 			<origin xyz="0 0 0.325" rpy="0 0 ${-PI/2}"/>
 		</joint>
+		<link name="camera_optical_frame"/>
+		<joint name="camera_sensor_pose_joint" type="fixed">
+			<parent link="camera_link"/>
+			<child link="camera_optical_frame"/>
+			<origin xyz="0 0 0" rpy="0 0 0"/>
+		</joint>
 	</xacro:macro>
 </robot>
